File: Robot Schematic/Robot.kicad_sch (KiCad schematic)
At the start: 15 parts, among them J1 Conn_01x04, J2 Conn_01x04, J3 Battery, J4 Switch, J5 Conn_01x06, J6 Conn_01x06, J7 Conn_01x06, U1 mp1584EN

Commit message: Add DWM Code, Add Transmitter Schematic/PCB
DWM Code features a new library that works and is tested with basic features
Parts:
- added C3, C4: 0.1uF, Capacitor_SMD:C_0805_2012Metric, symbol Device:C
- C1: value 100nF -> 0.1uF
- DWM1: MPN (none) -> DWM3000.E1.1SR
Connections:
- net +12V: now also C3.1, C4.1
- net GND: now also C3.2, C4.2
